Commit message: Got Cassie robot trained to walk, but kind of shuffles for FF model and hops for LSTM 16 model, I need to spend more time varying the reward hyperparameters, etc, to get useable/natural performance.

File: assets/urdf/cassie/urdf/cassie.urdf (robot description, URDF)
Before this commit: robot cassie, 16 links, 15 joints
Links:
- link left_toe: geometry collision mesh filename=../meshes/toe.stl scale=1 1 1; visual mesh filename=../meshes/toe.stl scale=1 1 1
- link right_toe: geometry collision mesh filename=../meshes/toe_mirror.stl scale=1 1 1; visual mesh filename=../meshes/toe_mirror.stl scale=1 1 1
Joints:
- joint toe_joint_right: limit lower=-2.4435 upper=-0.5236 effort=45 velocity=20.5192 -> lower=-2.4435 upper=0.5236 effort=45 velocity=20.5192
