Commit message: Anymal 0.5MASS-LSTM16-TERR works! 3 fixed points too. Tried 2.0MASS but that wasn't training very well, too slow. Going to retry A1 LSTM4 (with only zero ih_l0 bias), and also LSTM16 (with zero ih_l0 bias, hh_l0 bias, action_fb) with reward scale tuning.

File: assets/urdf/anymal_c/urdf/anymal_minimal_0pt5MASS.urdf (robot description, URDF)
Before this commit: robot anymal, 76 links, 75 joints
Links:
- link LF_FOOT: mass 0.21663 -> 0.108315
- link LF_HAA: mass 1.89871 -> 0.949355
- link LF_HFE: mass 1.89871 -> 0.949355
- link LF_HIP: mass 0.001 -> 0.0005
- link LF_KFE: mass 1.89871 -> 0.949355
- link LF_SHANK: mass 0.001 -> 0.0005
- link LF_THIGH: mass 0.001 -> 0.0005
- link LF_hip_fixed: mass 0.61232 -> 0.30616
- link LF_shank_fixed: mass 0.33742 -> 0.16871
- link LF_thigh_fixed: mass 1.37356 -> 0.68678
- link LH_FOOT: mass 0.21663 -> 0.108315
- link LH_HAA: mass 1.89871 -> 0.949355
- link LH_HFE: mass 1.89871 -> 0.949355
- link LH_HIP: mass 0.001 -> 0.0005
- link LH_KFE: mass 1.89871 -> 0.949355
- link LH_SHANK: mass 0.001 -> 0.0005
- link LH_THIGH: mass 0.001 -> 0.0005
- link LH_hip_fixed: mass 0.61232 -> 0.30616
- link LH_shank_fixed: mass 0.33742 -> 0.16871
- link LH_thigh_fixed: mass 1.37356 -> 0.68678
- link RF_FOOT: mass 0.21663 -> 0.108315
- link RF_HAA: mass 1.89871 -> 0.949355
- link RF_HFE: mass 1.89871 -> 0.949355
- link RF_HIP: mass 0.001 -> 0.0005
- link RF_KFE: mass 1.89871 -> 0.949355
- link RF_SHANK: mass 0.001 -> 0.0005
- link RF_THIGH: mass 0.001 -> 0.0005
- link RF_hip_fixed: mass 0.61232 -> 0.30616
- link RF_shank_fixed: mass 0.33742 -> 0.16871
- link RF_thigh_fixed: mass 1.37356 -> 0.68678
- link RH_FOOT: mass 0.21663 -> 0.108315
- link RH_HAA: mass 1.89871 -> 0.949355
- link RH_HFE: mass 1.89871 -> 0.949355
- link RH_HIP: mass 0.001 -> 0.0005
- link RH_KFE: mass 1.89871 -> 0.949355
- link RH_SHANK: mass 0.001 -> 0.0005
- link RH_THIGH: mass 0.001 -> 0.0005
- link RH_hip_fixed: mass 0.61232 -> 0.30616
- link RH_shank_fixed: mass 0.33742 -> 0.16871
- link RH_thigh_fixed: mass 1.37356 -> 0.68678
- link base: mass 10.3961 -> 5.19805
- link battery: mass 5.53425 -> 2.767125
- link blackfly_front_camera: mass 0.1716 -> 0.0858
- link blackfly_rear_camera: mass 0.1716 -> 0.0858
- link bottom_shell: mass 1.13247 -> 0.566235
- link face_front: mass 0.07792 -> 0.03896
- link face_rear: mass 0.07792 -> 0.03896
- link handle: mass 0.30655 -> 0.153275
- link hatch: mass 0.142 -> 0.071
- link imu_link: mass 0.01 -> 0.005
- link realsense_d435_front_camera: mass 0.10006 -> 0.05003
- link realsense_d435_left_camera: mass 0.10006 -> 0.05003
- link realsense_d435_rear_camera: mass 0.10006 -> 0.05003
- link realsense_d435_right_camera: mass 0.10006 -> 0.05003
- link top_shell: mass 0.602 -> 0.301
- link velodyne: mass 0.59 -> 0.295
- link velodyne_cage: mass 0.59537 -> 0.297685
