Commit message: Got A1Terrain model trained up (zero bias and fb) whoot! However, it has a weird asymmetric gait, and I suspect it has to do with the airtime, so I might try to tune that. Let's see what I can do.

File: assets/urdf/a1/urdf/a1.urdf (robot description, URDF)
Before this commit: robot a1_description, 23 links, 22 joints
Links:
- link trunk: geometry collision box size=0.497 0.194 0.114; visual mesh filename=../meshes/trunk.dae scale=1 1 1
